File: badge2.brd (EAGLE design)
At the start: 128 x 81 mm, 322 parts, among them IC1 LPC4330FET180, IC14 AT45DB041D, IC15 MCP73833, IC17 MAX15101EWL, IC18 MAX15101EWL, IC4 74AC04D, IC6 MAX2837ETM+, J2 U.FL, SW2 JS102011SAQN, X2 MICROUSB, X3 NOKIA

Commit message: Start with the RF-Layout
Place the components and change the rf-switches to get a good route
Parts:
- added IC8: 74AC04D, 74xx-eu:SO14
- moved U$10 380.1 mm to (-36.1, 67.6)
- moved U$13 368.7 mm to (-38.1, 64.5), turned to 180 degrees
- moved IC7 268.3 mm to (-47.8, 58.4)
- moved U$9 259.0 mm to (-35.3, 64.5)
- moved U$12 245.1 mm to (-37.3, 66.3), turned to 180 degrees
- moved U$11 241.3 mm to (-57.4, 63.2), turned to 180 degrees
- moved U$8 211.7 mm to (-56.1, 63.0), turned to 90 degrees
- moved U$7 196.4 mm to (-34.0, 64.5), turned to 180 degrees
- moved C220 176.2 mm to (-43.2, 65.3), turned to 180 degrees
- moved L12 175.2 mm to (-50.5, 66.3), turned to 270 degrees
- moved L11 174.9 mm to (-50.5, 63.2), turned to 90 degrees
- moved C225 174.1 mm to (-52.6, 65.3)
- moved C221 172.8 mm to (-43.2, 64.3), turned to 180 degrees
- moved U$6 172.3 mm to (-35.1, 71.6), turned to 180 degrees
- moved C222 171.6 mm to (-41.7, 64.8), turned to 90 degrees
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Connections:
- new net LOW_HIGH_FILT_N: IC4.6, U$7.6
- new net MIX_BY_N: IC8.8, U$11.6, U$12.6
- net AGND: now also U$13.2
- net BYPASS_RX: now also U$11.3; no longer U$11.1
- net GND: now also IC8.7; no longer U$13.2
- net LOW_HIGH_FILT: now also IC4.5; no longer U$7.6
- net MIX_BY: now also IC8.9; no longer U$11.6, U$12.6
- net N$10: now also FL2.1; no longer FL1.OUT
- net N$104: now also C225.1; no longer L9.4
- net N$109: now also L9.1; no longer C225.1
- net N$11: now also U$12.1; no longer U$12.3
- net N$110: now also L9.4; no longer L9.1
- net N$16: now also U$11.1; no longer U$11.3
- net N$4: now also U$12.3; no longer U$12.1
- net N$9: now also FL1.OUT; no longer FL2.1
- net VCC: now also IC8.14
Routing:
- net N$17: track 0.00 -> 35.4 mm
- net BYPASS_RX: track 0.00 -> 24.3 mm
- net N$10: track 0.00 -> 9.44 mm
- net N$38: track 0.00 -> 8.40 mm
- net N$19: track 0.00 -> 7.10 mm
- net AGND: track 0.00 -> 3.94 mm
- net N$9: track 0.00 -> 3.66 mm
- net BYPASS: track 0.00 -> 3.56 mm
- net N$5: track 0.00 -> 3.37 mm
- net N$15: track 0.00 -> 2.73 mm
- net N$32: track 0.00 -> 2.25 mm
- net N$8: track 0.00 -> 2.09 mm
- net N$6: track 0.00 -> 2.04 mm
- net N$105: track 0.00 -> 2.03 mm
- net N$36: track 0.00 -> 1.79 mm
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